Commit message: compensate leg height

File: carbodrone_px/models/x500/model.urdf (robot description, URDF)
Before this commit: robot x500, 4 links, 3 joints
Links:
- added link base_footprint
Joints:
- added joint base_footprint_joint: type fixed, parent base_link, child base_footprint, origin xyz=0 0 -0.23 rpy=0 0 0
